File: buttonbar/buttonbar.kicad_sch (KiCad schematic)
At the start: 44 parts, among them J1 Conn_01x08_Male, J2 Conn_01x06_Male, SW1 SW_Push, SW2 SW_Push, SW3 SW_Push, SW4 SW_Push, SW5 SW_Push, SW6 SW_Push, U1 74HC14D

Commit message: Rev 2.1
Parts:
- removed J1: Conn_01x08_Male, Connector_PinHeader_2.54mm:PinHeader_1x08_P2.54mm_Vertical, symbol Connector:Conn_01x08_Male
- added J1, J3: Conn_01x04_Male, Connector_PinHeader_2.54mm:PinHeader_1x04_P2.54mm_Vertical, symbol Connector:Conn_01x04_Male
- R13, R14, R15, R16, R17, R18: value 680 1206 -> 680 0603; footprint Resistor_SMD:R_1206_3216Metric_Pad1.30x1.75mm_HandSolder -> Resistor_SMD:R_0603_1608Metric; LCSC (none) -> C23212
- SW1, SW2, SW3, SW4, SW5, SW6: footprint user:SW_PUSH-6.12mm -> user:SW_PUSH_5.08mm
Connections:
- net BTN_1: now also J1.2 (Pin_2)
- net BTN_2: now also J1.3 (Pin_3)
- net BTN_3: now also J1.4 (Pin_4)
- net BTN_4: now also U1.8, J3.2 (Pin_2); no longer U1.12
- net BTN_5: now also J3.3 (Pin_3)
- net BTN_6: now also U1.12, J3.4 (Pin_4); no longer U1.8
- net GND: now also J1.1 (Pin_1)
- net Vcc: now also J3.1 (Pin_1)
- net at C4.1, R8.1: now also U1.9; no longer U1.13
- net at C6.1, R12.1: now also U1.13; no longer U1.9
Other:
- moved on the sheet: U1D, U1F

Commit message: Rev 2.2 (in production)
Parts:
- added H5, H6: MountingHole, MountingHole:MountingHole_2.5mm, symbol Mechanical:MountingHole
- D1, D2, D3, D4, D5, D6, H1, H2, H3, H4, J1, J2, J3, SW1, SW2, SW3, SW4, SW5, SW6: now left out of the parts list
Changed lines of the file:
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@@
   (title_block
     (title "PCB Buttonbar")
-    (date "2023-02-10")
-    (rev "2.1")
+    (date "2023-02-11")
+    (rev "2.2")
     (company "Bernhard Bablok")
     (comment 1 "https://github.com/bablokb/pcb-buttonbar")
@@
   )
   (symbol (lib_id "Switch:SW_Push") (at 33.02 38.1 0) (unit 1)
-    (in_bom yes) (on_board yes)
+    (in_bom no) (on_board yes)
     (property "Reference" "SW1" (id 0) (at 33.02 41.91 0))
     (property "Value" "SW_Push" (id 1) (at 33.02 44.45 0))
@@
   )
   (symbol (lib_id "Device:LED") (at 227.33 105.41 180) (unit 1)
-    (in_bom yes) (on_board yes)
+    (in_bom no) (on_board yes)
     (property "Reference" "D2" (id 0) (at 227.5078 98.933 0))
     (property "Value" "LED green 1206" (id 1) (at 227.5078 101.2444 0))
@@
   )
   (symbol (lib_id "Connector:Conn_01x06_Male") (at 186.69 121.92 0) (unit 1)
-    (in_bom yes) (on_board yes)
+    (in_bom no) (on_board yes)
     (property "Reference" "J2" (id 0) (at 187.96 107.95 0))
     (property "Value" "Conn_01x06_Male" (id 1) (at 187.96 111.76 0))
@@
   )
   (symbol (lib_id "Device:LED") (at 227.33 116.84 180) (unit 1)
-    (in_bom yes) (on_board yes)
+    (in_bom no) (on_board yes)
     (property "Reference" "D3" (id 0) (at 227.5078 110.363 0))
     (property "Value" "LED green 1206" (id 1) (at 227.5078 112.6744 0))
@@
   )
   (symbol (lib_id "Device:LED") (at 227.33 127 180) (unit 1)
-    (in_bom yes) (on_board yes)
+    (in_bom no) (on_board yes)
     (property "Reference" "D4" (id 0) (at 227.5078 120.523 0))
     (property "Value" "LED green 1206" (id 1) (at 227.5078 122.8344 0))
@@
   )
   (symbol (lib_id "Switch:SW_Push") (at 106.68 38.1 0) (unit 1)
-    (in_bom yes) (on_board yes)
+    (in_bom no) (on_board yes)
     (property "Reference" "SW2" (id 0) (at 106.68 40.64 0))
     (property "Value" "SW_Push" (id 1) (at 106.68 43.18 0))
@@
   )
   (symbol (lib_id "Device:LED") (at 227.33 138.43 180) (unit 1)
-    (in_bom yes) (on_board yes)
+    (in_bom no) (on_board yes)
     (property "Reference" "D5" (id 0) (at 227.5078 131.953 0))
     (property "Value" "LED green 1206" (id 1) (at 227.5078 134.2644 0))
@@
   )
   (symbol (lib_id "Device:LED") (at 227.33 149.86 180) (unit 1)
-    (in_bom yes) (on_board yes)
+    (in_bom no) (on_board yes)
     (property "Reference" "D6" (id 0) (at 227.5078 143.383 0))
     (property "Value" "LED green 1206" (id 1) (at 227.5078 145.6944 0))
@@
   )
   (symbol (lib_id "Device:LED") (at 227.33 95.25 180) (unit 1)
-    (in_bom yes) (on_board yes)
+    (in_bom no) (on_board yes)
     (property "Reference" "D1" (id 0) (at 227.5078 88.773 0))
     (property "Value" "LED green 1206" (id 1) (at 227.5078 91.0844 0))
@@
   )
   (symbol (lib_id "Switch:SW_Push") (at 33.02 82.55 0) (unit 1)
-    (in_bom yes) (on_board yes)
+    (in_bom no) (on_board yes)
     (property "Reference" "SW3" (id 0) (at 33.02 86.36 0))
     (property "Value" "SW_Push" (id 1) (at 33.02 88.9 0))
@@
   )
   (symbol (lib_id "Switch:SW_Push") (at 106.68 82.55 0) (unit 1)
-    (in_bom yes) (on_board yes)
+    (in_bom no) (on_board yes)
     (property "Reference" "SW4" (id 0) (at 106.68 86.36 0))
     (property "Value" "SW_Push" (id 1) (at 106.68 88.9 0))
@@
   )
   (symbol (lib_id "Switch:SW_Push") (at 33.02 127 0) (unit 1)
-    (in_bom yes) (on_board yes)
+    (in_bom no) (on_board yes)
     (property "Reference" "SW5" (id 0) (at 34.29 130.81 0))
     (property "Value" "SW_Push" (id 1) (at 34.29 133.35 0))
@@
   )
   (symbol (lib_id "Switch:SW_Push") (at 106.68 127 0) (unit 1)
-    (in_bom yes) (on_board yes)
+    (in_bom no) (on_board yes)
     (property "Reference" "SW6" (id 0) (at 106.68 130.81 0))
     (property "Value" "SW_Push" (id 1) (at 106.68 134.62 0))
@@
   )
   (symbol (lib_id "Mechanical:MountingHole") (at 116.84 182.88 0) (unit 1)
-    (in_bom yes) (on_board yes)
+    (in_bom no) (on_board yes)
     (property "Reference" "H3" (id 0) (at 119.38 181.7116 0)
       (effects (font (size 1.27 1.27)) (justify left))
@@
   )
   (symbol (lib_id "Mechanical:MountingHole") (at 116.84 175.26 0) (unit 1)
-    (in_bom yes) (on_board yes)
+    (in_bom no) (on_board yes)
     (property "Reference" "H1" (id 0) (at 119.38 174.0916 0)
       (effects (font (size 1.27 1.27)) (justify left))
@@
   )
   (symbol (lib_id "Mechanical:MountingHole") (at 144.78 175.26 0) (unit 1)
-    (in_bom yes) (on_board yes)
+    (in_bom no) (on_board yes)
     (property "Reference" "H2" (id 0) (at 147.32 174.0916 0)
       (effects (font (size 1.27 1.27)) (justify left))
@@
   )
   (symbol (lib_id "Mechanical:MountingHole") (at 144.78 184.15 0) (unit 1)
-    (in_bom yes) (on_board yes)
+    (in_bom no) (on_board yes)
     (property "Reference" "H4" (id 0) (at 147.32 182.9816 0)
       (effects (font (size 1.27 1.27)) (justify left))
@@
     )
     (property "Datasheet" "~" (id 3) (at 144.78 184.15 0)
+      (effects (font (size 1.27 1.27)) hide)
+    )
+  )
+  (symbol (lib_id "Mechanical:MountingHole") (at 117.475 191.135 0) (unit 1)
+    (in_bom no) (on_board yes)
+    (property "Reference" "H5" (id 0) (at 120.015 189.9666 0)
+      (effects (font (size 1.27 1.27)) (justify left))
+    )
+    (property "Value" "MountingHole" (id 1) (at 120.015 192.278 0)
+      (effects (font (size 1.27 1.27)) (justify left))
+    )
+    (property "Footprint" "MountingHole:MountingHole_2.5mm" (id 2) (at 117.475 191.135 0)
+      (effects (font (size 1.27 1.27)) hide)
+    )
+    (property "Datasheet" "~" (id 3) (at 117.475 191.135 0)
       (effects (font (size 1.27 1.27)) hide)
     )
@@
   )
   (symbol (lib_id "Connector:Conn_01x04_Male") (at 184.15 66.04 0) (unit 1)
-    (in_bom yes) (on_board yes)
+    (in_bom no) (on_board yes)
     (property "Reference" "J3" (id 0) (at 172.72 64.135 0))
     (property "Value" "Conn_01x04_Male" (id 1) (at 172.72 66.675 0))
@@
     (pin "4")
   )
+  (symbol (lib_id "Mechanical:MountingHole") (at 145.415 192.405 0) (unit 1)
+    (in_bom no) (on_board yes)
+    (property "Reference" "H6" (id 0) (at 147.955 191.2366 0)
+      (effects (font (size 1.27 1.27)) (justify left))
+    )
+    (property "Value" "MountingHole" (id 1) (at 147.955 193.548 0)
+      (effects (font (size 1.27 1.27)) (justify left))
+    )
+    (property "Footprint" "MountingHole:MountingHole_2.5mm" (id 2) (at 145.415 192.405 0)
+      (effects (font (size 1.27 1.27)) hide)
+    )
+    (property "Datasheet" "~" (id 3) (at 145.415 192.405 0)
+      (effects (font (size 1.27 1.27)) hide)
+    )
+  )
   (symbol (lib_id "Connector:Conn_01x04_Male") (at 184.15 55.88 0) (unit 1)
-    (in_bom yes) (on_board yes)
+    (in_bom no) (on_board yes)
     (property "Reference" "J1" (id 0) (at 172.72 53.34 0))
     (property "Value" "Conn_01x04_Male" (id 1) (at 172.72 57.15 0))
@@
       (reference "H4") (unit 1) (value "MountingHole") (footprint "MountingHole:MountingHole_2.5mm")
     )
+    (path "/2a5410b2-8875-4f19-8aee-8df23f4d99d3"
+      (reference "H5") (unit 1) (value "MountingHole") (footprint "MountingHole:MountingHole_2.5mm")
+    )
+    (path "/f5d39a21-bfa6-4eed-bb3d-07b95ee461d4"
+      (reference "H6") (unit 1) (value "MountingHole") (footprint "MountingHole:MountingHole_2.5mm")
+    )
     (path "/fe1d719b-36e2-4a79-aeb0-6270f4520f52"
